File: cpu-board/z80-cpu-dip.kicad_pcb (KiCad board)
At the start: 2 copper layers, 34 parts, among them IC1 Z84C0006, IC2 Z8470, J1 PWR, J2 SER0, J3 D/C, J4 IO, Q1 2N3904, U1 AT28C64B-15PU, U10 74LS373, U11 74LS32, U12 SN74HC14N, U2 74LS373, U3 KM62256CLP, U4 74LS08, U5 74LS139, U6 KM62256CLP, U7 74LS154, U8 SN74HC14N, U9 SN74HC14N, X1 CXO_DIP14

Commit message: Updated PCB and SCH
Parts:
- moved R2 54.2 mm to (190.7, 116.6)
- moved D6 54.2 mm to (198.3, 105.8)
- moved J2 54.2 mm to (206.6, 85.1)
- moved Q1 54.2 mm to (197.0, 80.6)
- moved R3 54.2 mm to (200.8, 91.8)
- moved U12 54.2 mm to (60.5, 128.3)
- moved D4 54.2 mm to (198.3, 99.4)
- moved D7 54.2 mm to (198.3, 108.9)
- moved IC1 54.2 mm to (60.5, 116.8)
- moved IC2 54.2 mm to (60.5, 97.8)
- moved J1 54.2 mm to (206.6, 72.4)
- moved J3 54.2 mm to (55.4, 64.1)
- moved J4 54.2 mm to (55.4, 117.5)
- moved R1 54.2 mm to (190.7, 112.7)
- moved RN1 54.2 mm to (108.8, 78.1)
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Routing:
- net BANK2 SEL*: track 141.9 -> 56.5 mm, vias 1 -> 0
- net IO6*: track 253.7 -> 174.7 mm, vias 4 -> 9
- net IO3*: track 217.5 -> 154.3 mm, vias 2 -> 3
- net IO1*: track 212.8 -> 153.7 mm, vias 2 -> 5
- net Net-(U11-Pad5): track 145.4 -> 91.3 mm, vias 6 -> 0
- net A2: track 160.6 -> 213.1 mm, vias 1 -> 2
- net OB LED: track 130.3 -> 79.3 mm, vias 5 -> 0
- net RESET*: track 251.0 -> 212.5 mm, vias 3 -> 2
- net ROM*/RAM: track 249.8 -> 215.0 mm, vias 3 -> 4
- net A15: track 89.3 -> 58.0 mm, vias 1 -> 2
- net BANK3 SEL: track 101.3 -> 70.6 mm, vias 3 -> 2
- net BANK3 SEL*: track 94.4 -> 121.9 mm, vias 2 -> 6
- net ROM SEL*: track 33.9 -> 61.4 mm, vias 0 -> 3
- net DART SEL*: track 153.7 -> 127.1 mm, vias 3 -> 1
- net RESET: track 261.8 -> 235.5 mm
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Other:
- board outline added: 162.6 x 71.1 mm
